Commit message: feat: 관측 기반 경로 계획 고도화 및 기본 주행 프로파일 적용
- Hybrid A* + RPP를 기본 플래닝 조합으로 적용
- 관측 통로 기반 경유점 선택과 다중 비용 경로 탐색 추가
- 미관측 영역 진입 검사와 관측 방향 회전 검사 적용
- 기존 경로 유지 및 경유점 도달 가능성 재검사 추가
- 최종 목표 접근 시 목표 고정과 정지·재계획 정책 적용
- 인지 지도 처리와 의미분할 지연 진단 기능 보강
- ZED 2 근사 센서 설정 및 VIO 보정 설정 반영
- Map04 B0 모델과 플래닝 실험 도구 및 회귀 테스트 추가

File: src/nomad_gazebo/urdf/nomad_vehicle.urdf (robot description, URDF)
Before this commit: robot nomad_vehicle, 13 links, 12 joints
Joints:
- joint oak_left_optical_frame_joint: origin xyz=0.46 0.0375 0.29 rpy=-1.5707963267949 0 -1.5707963267949 -> xyz=0.46 0.06 0.29 rpy=-1.5707963267949 0 -1.5707963267949
- joint oak_right_optical_frame_joint: origin xyz=0.46 -0.0375 0.29 rpy=-1.5707963267949 0 -1.5707963267949 -> xyz=0.46 -0.06 0.29 rpy=-1.5707963267949 0 -1.5707963267949

Commit message: feat: 전륜 구동·후륜 조향과 통합 주행 구조 적용

File: src/nomad_gazebo/urdf/nomad_vehicle.urdf (robot description, URDF)
Before this commit: robot nomad_vehicle, 13 links, 12 joints
Links:
- removed link front_left_steering_link
- removed link front_right_steering_link
- added link rear_left_steering_link, mass 0.3; visual cylinder length=0.04 radius=0.025
- added link rear_right_steering_link, mass 0.3; visual cylinder length=0.04 radius=0.025
Joints:
- removed joint front_left_steering_joint
- removed joint front_right_steering_joint
- added joint rear_left_steering_joint: type revolute, parent base_link, child rear_left_steering_link, origin xyz=-0.36 0.3 0.15 rpy=0 0 0, axis 0 0 1, limit lower=-0.55 upper=0.55 effort=12 velocity=2
- added joint rear_right_steering_joint: type revolute, parent base_link, child rear_right_steering_link, origin xyz=-0.36 -0.3 0.15 rpy=0 0 0, axis 0 0 1, limit lower=-0.55 upper=0.55 effort=12 velocity=2
- joint front_left_wheel_joint: origin xyz=0 0 0 rpy=0 0 0 -> xyz=0.36 0.3 0.15 rpy=0 0 0; parent front_left_steering_link -> base_link
- joint front_right_wheel_joint: origin xyz=0 0 0 rpy=0 0 0 -> xyz=0.36 -0.3 0.15 rpy=0 0 0; parent front_right_steering_link -> base_link
- joint rear_left_wheel_joint: origin xyz=-0.36 0.3 0.15 rpy=0 0 0 -> xyz=0 0 0 rpy=0 0 0; parent base_link -> rear_left_steering_link
- joint rear_right_wheel_joint: origin xyz=-0.36 -0.3 0.15 rpy=0 0 0 -> xyz=0 0 0 rpy=0 0 0; parent base_link -> rear_right_steering_link
